Commit message: add pgc arm

File: dobot_description/urdf/nova2_robot.urdf (robot description, URDF)
Before this commit: robot nova2_robot, 8 links, 7 joints
Links:
- added link finger1_link, mass 0.014278; collision mesh filename=package://dh_pgc140_urdf/meshes/finger1_Link.STL; visual mesh filename=package://dh_pgc140_urdf/meshes/finger1_Link.STL
- added link finger2_link, mass 0.014278; collision mesh filename=package://dh_pgc140_urdf/meshes/finger2_Link.STL; visual mesh filename=package://dh_pgc140_urdf/meshes/finger2_Link.STL
- added link hand_base_link, mass 0.34365; collision mesh filename=package://dh_pgc140_urdf/meshes/base_link.STL; visual mesh filename=package://dh_pgc140_urdf/meshes/base_link.STL
Joints:
- added joint endeffect: type prismatic, parent Link6, child hand_base_link, origin xyz=0.0 0.0 0.007 rpy=0 0 0, axis 1 0 0, limit lower=0 upper=0.025 effort=140 velocity=1
- added joint finger1_joint: type prismatic, parent hand_base_link, child finger1_link, origin xyz=0.0132 0.0265 0.093 rpy=0 0 -1.5708, axis 1 0 0, limit lower=0 upper=0.025 effort=140 velocity=1
- added joint finger2_joint: type prismatic, parent hand_base_link, child finger2_link, origin xyz=-0.0132 -0.0265 0.093 rpy=0 0 1.5708, axis 1 0 0, limit lower=0 upper=0.025 effort=140 velocity=1, mimic joint=finger1_joint multiplier=1 offset=0

Commit message: update to simple collision

File: dobot_description/urdf/nova2_robot.urdf (robot description, URDF)
Before this commit: robot nova2_robot, 11 links, 10 joints
Links:
- link finger1_link: geometry collision box size=0.01 0.01 0.03; visual mesh filename=package://dh_pgc140_urdf/meshes/finger1_Link.STL
- link finger2_link: geometry collision box size=0.01 0.01 0.03; visual mesh filename=package://dh_pgc140_urdf/meshes/finger2_Link.STL
- link hand_base_link: geometry collision box size=0.063 0.063 0.099; visual mesh filename=package://dh_pgc140_urdf/meshes/base_link.STL
Joints:
- joint endeffect: axis 1 0 0 -> (none); limit lower=0 upper=0.025 effort=140 velocity=1 -> (none); origin xyz=0.0 0.0 0.007 rpy=0 0 0 -> xyz=0.0 0.0 0.0 rpy=0 0 0; type prismatic -> fixed

Commit message: replace gripper urdf

File: dobot_description/urdf/nova2_robot.urdf (robot description, URDF)
Before this commit: robot nova2_robot, 11 links, 10 joints
Links:
- link finger1_link: geometry collision box size=0.01 0.01 0.03; visual mesh filename=package://dobot_description/meshes/nova2/finger/finger1_Lin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
- link finger2_link: geometry collision box size=0.01 0.01 0.03; visual mesh filename=package://dobot_description/meshes/nova2/finger/finger2_Lin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
- link hand_base_link: geometry collision box size=0.063 0.063 0.099; visual mesh filename=package://dobot_description/meshes/nova2/finger/base_link.S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

Commit message: tested real robot

File: dobot_description/urdf/nova2_robot.urdf (robot description, URDF)
Before this commit: robot nova2_robot, 11 links, 10 joints
Links:
- link finger1_link: geometry collision cylinder length=0.04 radius=0.01; visual mesh filename=package://dobot_description/meshes/nova2/finger/finger1_Lin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
- link finger2_link: geometry collision cylinder length=0.04 radius=0.01; visual mesh filename=package://dobot_description/meshes/nova2/finger/finger2_Lin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
- link hand_base_link: geometry collision cylinder length=0.08 radius=0.04; visual mesh filename=package://dobot_description/meshes/nova2/finger/base_link.S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
Joints:
- removed joint endeffect
- added joint joint7: type fixed, parent Link6, child hand_base_link, origin xyz=0.0 0.0 0.0 rpy=0 0 0
- joint joint6: limit lower=-6.28 upper=6.28 effort=0 velocity=0 -> lower=-3.13 upper=3.13 effort=0 velocity=0

Commit message: make bigger cylnder

File: dobot_description/urdf/nova2_robot.urdf (robot description, URDF)
Before this commit: robot nova2_robot, 11 links, 10 joints
Links:
- link hand_base_link: geometry collision cylinder length=0.13 radius=0.06; visual mesh filename=package://dobot_description/meshes/nova2/finger/base_link.S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

Commit message: add camera

File: dobot_description/urdf/nova2_robot.urdf (robot description, URDF)
Before this commit: robot nova2_robot, 11 links, 10 joints
Links:
- added link camera, mass 0.34365; collision box size=0.06 0.05 0.03; visual box size=0.06 0.05 0.03
Joints:
- added joint joint8: type fixed, parent Link6, child camera, origin xyz=0.0 0.0 0.0 rpy=0 0 0

Commit message: update collision

File: dobot_description/urdf/nova2_robot.urdf (robot description, URDF)
Before this commit: robot nova2_robot, 12 links, 11 joints
Links:
- link camera: geometry collision box size=0.05 0.06 0.03; visual box size=0.05 0.06 0.03
- link hand_base_link: geometry collision cylinder length=0.13 radius=0.053; visual mesh filename=package://dobot_description/meshes/nova2/finger/base_link.S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
Joints:
- joint joint8: parent Link6 -> hand_base_link
